Commit message: 更新大人形URDF

File: source/unitree_rl_lab/unitree_rl_lab/assets/robots/humanoid_ultra_description/urdf/humanoidultra12dof_mpc.urdf (robot description, URDF)
Before this commit: robot humanoidultra01, 28 links, 27 joints
Links:
- added link dummy_link
- added link l_foot_heel
- added link l_foot_toe
- added link r_foot_heel
- added link r_foot_toe
- link base_link: geometry collision box size=0.114 0.405 0.06235863854; collision box size=0.15 0.26 0.01
- link left_ankle_pitch_link: geometry visual mesh filename=package://humanoidultra_urdf/meshes/left_ankle_pitch_link.S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
- link left_ankle_roll_link: geometry collision cylinder length=0.099745 radius=0.003; collision cylinder length=0.099745 radius=0.003
- link left_elbow_link: geometry visual mesh filename=package://humanoidultra_urdf/meshes/left_elbow_link.STL
- link left_hip_pitch_link: geometry collision box size=0.05 0.049 0.36; collision sphere radius=0.085
- link left_hip_roll_link: geometry visual mesh filename=package://humanoidultra_urdf/meshes/left_hip_roll_link.STL
- link left_hip_yaw_link: geometry visual mesh filename=package://humanoidultra_urdf/meshes/left_hip_yaw_link.STL
- link left_knee_link: geometry collision box size=0.05 0.027 0.26; visual mesh filename=package://humanoidultra_urdf/meshes/left_knee_link.STL
- link left_shoulder_pitch_link: geometry collision cylinder length=0.076 radius=0.033; visual mesh filename=package://humanoidultra_urdf/meshes/left_shoulder_pitch_lin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
- link left_shoulder_roll_link: geometry visual mesh filename=package://humanoidultra_urdf/meshes/left_shoulder_roll_link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
- link left_shoulder_yaw_link: geometry collision box size=0.05 0.05 0.081; visual mesh filename=package://humanoidultra_urdf/meshes/left_shoulder_yaw_link.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
- link left_wrist_pitch_link: geometry visual mesh filename=package://humanoidultra_urdf/meshes/left_wrist_pitch_link.S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
- link left_wrist_roll_link: geometry visual mesh filename=package://humanoidultra_urdf/meshes/left_wrist_roll_link.STL
- link left_wrist_yaw_link: geometry collision cylinder length=0.071 radius=0.033; visual mesh filename=package://humanoidultra_urdf/meshes/left_wrist_yaw_link.STL
- link right_ankle_pitch_link: geometry visual mesh filename=package://humanoidultra_urdf/meshes/right_ankle_pitch_link.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
- link right_ankle_roll_link: geometry collision cylinder length=0.099745 radius=0.003; collision cylinder length=0.099745 radius=0.003
- link right_elbow_link: geometry visual mesh filename=package://humanoidultra_urdf/meshes/right_elbow_link.STL
- link right_hip_pitch_link: geometry collision box size=0.05 0.049 0.36; collision sphere radius=0.085
- link right_hip_roll_link: geometry visual mesh filename=package://humanoidultra_urdf/meshes/right_hip_roll_link.STL
- link right_hip_yaw_link: geometry visual mesh filename=package://humanoidultra_urdf/meshes/right_hip_yaw_link.STL
- link right_knee_link: geometry collision box size=0.05 0.027 0.26; visual mesh filename=package://humanoidultra_urdf/meshes/right_knee_link.STL
- link right_shoulder_pitch_link: geometry collision cylinder length=0.076 radius=0.033; visual mesh filename=package://humanoidultra_urdf/meshes/right_shoulder_pitch_li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
- link right_shoulder_roll_link: geometry visual mesh filename=package://humanoidultra_urdf/meshes/right_shoulder_roll_lin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
- link right_shoulder_yaw_link: geometry collision box size=0.05 0.05 0.081; visual mesh filename=package://humanoidultra_urdf/meshes/right_shoulder_yaw_link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
- link right_wrist_pitch_link: geometry visual mesh filename=package://humanoidultra_urdf/meshes/right_wrist_pitch_link.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
- link right_wrist_roll_link: geometry visual mesh filename=package://humanoidultra_urdf/meshes/right_wrist_roll_link.S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
- link right_wrist_yaw_link: geometry collision cylinder length=0.071 radius=0.033; visual mesh filename=package://humanoidultra_urdf/meshes/right_wrist_yaw_link.STL
- link trunk_link: geometry collision box size=0.108 0.06 0.201; collision box size=0.108 0.06 0.201
Joints:
- added joint dummy_to_base_link: type fixed, parent dummy_link, child base_link, origin xyz=0.115315 0.0 -0.015775 rpy=0 0 0
- added joint l_foot_heel_joint: type fixed, parent left_ankle_roll_link, child l_foot_heel, origin xyz=-0.07771537914 0.0 -0.0522964 rpy=0 0.0 0.0
- added joint l_foot_toe_joint: type fixed, parent left_ankle_roll_link, child l_foot_toe, origin xyz=0.130962573 0.0 -0.0522964 rpy=0 0.0 0.0
- added joint r_foot_heel_joint: type fixed, parent right_ankle_roll_link, child r_foot_heel, origin xyz=-0.07771537914 0.0 -0.0522964 rpy=0 0.0 0.0
- added joint r_foot_toe_joint: type fixed, parent right_ankle_roll_link, child r_foot_toe, origin xyz=0.130962573 0.0 -0.0522964 rpy=0 0.0 0.0
- joint left_elbow_joint: origin xyz=0 -0.00025881904510211 -0.151965925826289 rpy=0 0 0 -> xyz=0 -0.00025881904510211 -0.151965925826289 rpy=-1.04720 0 0; type revolute -> fixed
- joint left_shoulder_pitch_joint: origin xyz=0 0.128943749506644 0.352787572334531 rpy=0.261799387799149 0 0 -> xyz=0 0.128943749506644 0.352787572334531 rpy=0.28228151180682093 0.3786256514483699 0.1067984530673944; type revolute -> fixed
- joint left_shoulder_roll_joint: origin xyz=0 0.0630000000000002 0 rpy=-0.26179938779915 0 0 -> xyz=0 0.0630000000000002 0 rpy=-0.16179938779915 0 0; type revolute -> fixed
- joint left_shoulder_yaw_joint: origin xyz=0 0.065813 -0.091069 rpy=0.2618 0 0 -> xyz=0 0.065813 -0.091069 rpy=0 -0.2618 1.5708; type revolute -> fixed
- joint left_wrist_pitch_joint: type revolute -> fixed
- joint left_wrist_roll_joint: type revolute -> fixed
- joint left_wrist_yaw_joint: origin xyz=0 0 -0.0915 rpy=0 0 0 -> xyz=0 0 -0.0915 rpy=0 0 -1.5708; type revolute -> fixed
- joint right_elbow_joint: origin xyz=0 0.00025881904510261 -0.151965925826289 rpy=0 0 0 -> xyz=0 0.00025881904510261 -0.151965925826289 rpy=1.04720 0 0; type revolute -> fixed
- joint right_shoulder_pitch_joint: origin xyz=0 -0.128943749506644 0.352787572334531 rpy=-0.26179938779915 0 0 -> xyz=0 -0.128943749506644 0.352787572334531 rpy=-0.28228151180682093 0.3786256514483699 -0.1067984530673944; type revolute -> fixed
- joint right_shoulder_roll_joint: origin xyz=0 -0.063 0 rpy=0.26179938779915 0 0 -> xyz=0 -0.063 0 rpy=0.16179938779915 0 0; type revolute -> fixed
- joint right_shoulder_yaw_joint: origin xyz=0 -0.065813 -0.091069 rpy=-0.2618 0 0 -> xyz=0 -0.065813 -0.091069 rpy=0 -0.2618 -1.5708; type revolute -> fixed
- joint right_wrist_pitch_joint: type revolute -> fixed
- joint right_wrist_roll_joint: type revolute -> fixed
- joint right_wrist_yaw_joint: origin xyz=0 0 -0.0915 rpy=0 0 0 -> xyz=0 0 -0.0915 rpy=0 0 1.5708; type revolute -> fixed
- joint waist_yaw_joint: type revolute -> fixed

File: source/unitree_rl_lab/unitree_rl_lab/assets/robots/humanoid_ultra_description_0630/urdf/humanoid_ultra_12dof_description.urdf (robot description, URDF)
Before this commit: robot humanoidultra01, 28 links, 27 joints
Links:
- added link dummy_link
- added link l_foot_heel
- added link l_foot_toe
- added link left_knee_imu
- added link neck_pitch_link, mass 0.568971862007055; collision box size=0.06525 0.14363 0.10427; visual mesh filename=package://humanoid_ultra_description/meshes/neck_pitch_link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
- added link neck_yaw_link, mass 0.44388106; collision cylinder length=0.0566 radius=0.026; visual mesh filename=package://humanoid_ultra_description/meshes/neck_yaw_link.S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
- added link r_foot_heel
- added link r_foot_toe
- added link right_knee_imu
- link base_link: mass 7.87598286 -> 7.89106591706423; geometry collision box size=0.15 0.3 0.1; visual mesh filename=package://humanoid_ultra_description/meshes/base_link.STL
- link left_ankle_pitch_link: mass 0.05651532 -> 0.0241612944467329; geometry visual mesh filename=package://humanoid_ultra_description/meshes/left_ankle_pitc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
- link left_ankle_roll_link: mass 0.75938458 -> 0.828995344627804; geometry collision cylinder length=0.20267795214 radius=0.003; collision cylinder length=0.20267795214 radius=0.003
- link left_elbow_link: mass 0.53459108 -> 0.527226; geometry collision cylinder length=0.0585 radius=0.033; visual mesh filename=package://humanoid_ultra_description/meshes/left_elbow_link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
- link left_hip_pitch_link: mass 8.43224915 -> 8.35630276269156; geometry collision box size=0.05 0.049 0.36; collision cylinder length=0.045 radius=0.085
- link left_hip_roll_link: mass 1.58332093 -> 1.73664512071164; geometry collision box size=0.114 0.105 0.056; visual mesh filename=package://humanoid_ultra_description/meshes/left_hip_roll_l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
- link left_hip_yaw_link: mass 1.47113700 -> 1.46284235577634; geometry collision cylinder length=0.026 radius=0.0395; visual mesh filename=package://humanoid_ultra_description/meshes/left_hip_yaw_li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
- link left_knee_link: mass 2.20062290 -> 2.02536692124872; geometry collision box size=0.05 0.027 0.3; visual mesh filename=package://humanoid_ultra_description/meshes/left_knee_link.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
- link left_shoulder_pitch_link: mass 0.69960149 -> 0.674662; geometry collision cylinder length=0.076 radius=0.033; visual mesh filename=package://humanoid_ultra_description/meshes/left_shoulder_p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
- link left_shoulder_roll_link: mass 0.76368656 -> 0.752079; geometry visual mesh filename=package://humanoid_ultra_description/meshes/left_shoulder_r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
- link left_shoulder_yaw_link: mass 0.78058169 -> 0.755247; geometry collision box size=0.05 0.05 0.081; visual mesh filename=package://humanoid_ultra_description/meshes/left_shoulder_y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
- link left_wrist_pitch_link: mass 0.37464276 -> 0.611201; geometry visual mesh filename=package://humanoid_ultra_description/meshes/left_wrist_pitc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
- link left_wrist_roll_link: mass 0.61394363 -> 0.587201; geometry collision cylinder length=0.0695 radius=0.031; visual mesh filename=package://humanoid_ultra_description/meshes/left_wrist_roll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
- link left_wrist_yaw_link: mass 0.63301211 -> 0.616108; geometry collision cylinder length=0.071 radius=0.033; visual mesh filename=package://humanoid_ultra_description/meshes/left_wrist_yaw_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
- link right_ankle_pitch_link: mass 0.05651532 -> 0.0241612944467328; geometry visual mesh filename=package://humanoid_ultra_description/meshes/right_ankle_pit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
- link right_ankle_roll_link: mass 0.75938458 -> 0.828995344627804; geometry collision cylinder length=0.20267795214 radius=0.003; collision cylinder length=0.20267795214 radius=0.003
- link right_elbow_link: mass 0.53459108 -> 0.527226; geometry collision cylinder length=0.0585 radius=0.033; visual mesh filename=package://humanoid_ultra_description/meshes/right_elbow_lin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
- link right_hip_pitch_link: mass 8.45830779 -> 8.38236123080177; geometry collision box size=0.05 0.049 0.36; collision cylinder length=0.045 radius=0.085
- link right_hip_roll_link: mass 1.58332093 -> 1.73664512071165; geometry collision box size=0.114 0.105 0.056; visual mesh filename=package://humanoid_ultra_description/meshes/right_hip_roll_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
- link right_hip_yaw_link: mass 1.47113700 -> 1.46284235577635; geometry collision cylinder length=0.026 radius=0.0395; visual mesh filename=package://humanoid_ultra_description/meshes/right_hip_yaw_l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
- link right_knee_link: mass 2.21352893 -> 2.02536771173414; geometry collision box size=0.05 0.027 0.3; visual mesh filename=package://humanoid_ultra_description/meshes/right_knee_link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
- link right_shoulder_pitch_link: mass 0.69960149 -> 0.674662; geometry collision cylinder length=0.076 radius=0.033; visual mesh filename=package://humanoid_ultra_description/meshes/right_shoulder_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
- link right_shoulder_roll_link: mass 0.76368656 -> 0.752079; geometry visual mesh filename=package://humanoid_ultra_description/meshes/right_shoulder_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
- link right_shoulder_yaw_link: mass 0.78058104 -> 0.755247; geometry collision box size=0.05 0.05 0.081; visual mesh filename=package://humanoid_ultra_description/meshes/right_shoulder_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
- link right_wrist_pitch_link: mass 0.37464274 -> 0.611201; geometry visual mesh filename=package://humanoid_ultra_description/meshes/right_wrist_pit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
- link right_wrist_roll_link: mass 0.61737346 -> 0.587201; geometry collision cylinder length=0.0695 radius=0.031; visual mesh filename=package://humanoid_ultra_description/meshes/right_wrist_rol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
- link right_wrist_yaw_link: mass 0.63301211 -> 0.614736; geometry collision cylinder length=0.071 radius=0.033; visual mesh filename=package://humanoid_ultra_description/meshes/right_wrist_yaw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
- link trunk_link: mass 11.2484619397318 -> 12.364176; geometry collision box size=0.185 0.2655 0.201; visual mesh filename=package://humanoid_ultra_description/meshes/trunk_link.STL
Joints:
- added joint dummy_to_base_link: type fixed, parent dummy_link, child base_link, origin xyz=0.115315 0.0 -0.015775 rpy=0 0 0
- added joint l_foot_heel_joint: type fixed, parent left_ankle_roll_link, child l_foot_heel, origin xyz=-0.07771537914 0.0 -0.046568515 rpy=0 0.0 0.0
- added joint l_foot_toe_joint: type fixed, parent left_ankle_roll_link, child l_foot_toe, origin xyz=0.130962573 0.0 -0.046568515 rpy=0 0.0 0.0
- added joint left_knee_imu_joint: type fixed, parent left_knee_link, child left_knee_imu, origin xyz=0.0467 0.0 -0.0335 rpy=1.5708 0.0 1.5708
- added joint neck_pitch_joint: type fixed, parent neck_yaw_link, child neck_pitch_link, origin xyz=0 0 0.045 rpy=0 0 0, axis 0 -1 0, limit lower=-1.5707 upper=1.5707 effort=14.0 velocity=6.28
- added joint neck_yaw_joint: type fixed, parent trunk_link, child neck_yaw_link, origin xyz=0 0 0.4259 rpy=0 0 0, axis 0 0 1, limit lower=-2.618 upper=2.618 effort=12.0 velocity=12.0
- added joint r_foot_heel_joint: type fixed, parent right_ankle_roll_link, child r_foot_heel, origin xyz=-0.07771537914 0.0 -0.046568515 rpy=0 0.0 0.0
- added joint r_foot_toe_joint: type fixed, parent right_ankle_roll_link, child r_foot_toe, origin xyz=0.130962573 0.0 -0.046568515 rpy=0 0.0 0.0
- added joint right_knee_imu_joint: type fixed, parent right_knee_link, child right_knee_imu, origin xyz=0.0467 0.0 -0.0335 rpy=1.5708 0.0 1.5708
- joint left_ankle_pitch_joint: limit lower=-0.7 upper=0.95 effort=72 velocity=12.0 -> lower=-0.7 upper=0.95 effort=72.0 velocity=12.0; origin xyz=0.000178842126592992 0 -0.367370694199002 rpy=0 0 0 -> xyz=0 0 -0.3713667324878 rpy=0 0 0
- joint left_ankle_roll_joint: axis 0.996194698091745 0 -0.0871557427476591 -> 0.996194698091743 0 -0.0871557427476896; limit lower=-0.45 upper=0.45 effort=72 velocity=12.0 -> lower=-0.45 upper=0.45 effort=72.0 velocity=12.0
- joint left_elbow_joint: limit lower=-2.17 upper=0 effort=72 velocity=8.164 -> lower=-2.17 upper=0.0 effort=70.0 velocity=6.28; origin xyz=0 -0.00025881904510211 -0.151965925826289 rpy=-1.04720 0 0 -> xyz=0 0 -0.151 rpy=0 0 0
- joint left_hip_pitch_joint: limit lower=-1.57 upper=1.57 effort=320 velocity=12.0 -> lower=-1.5708 upper=1.5708 effort=320.0 velocity=12.0; origin xyz=0 -0.00680000000000071 -0.1652 rpy=0 0 0 -> xyz=0 -0.00679999999999965 -0.1652 rpy=0 0 0
- joint left_hip_roll_joint: limit lower=-0.25 upper=1.57 effort=300 velocity=12.0 -> lower=-0.1 upper=1.5708 effort=320.0 velocity=12.0
- joint left_hip_yaw_joint: limit lower=-1.57 upper=1.57 effort=90 velocity=12.0 -> lower=-1.5708 upper=1.5708 effort=90.0 velocity=12.0
- joint left_knee_joint: limit lower=0.0 upper=2.36 effort=320 velocity=12.0 -> lower=0.0 upper=2.356 effort=320.0 velocity=12.0; origin xyz=0 0 -0.38 rpy=0 0 0 -> xyz=0 0 -0.379999999999996 rpy=0 0 0
- joint left_shoulder_pitch_joint: limit lower=-2.4 upper=1.2 effort=72 velocity=8.164 -> lower=-2.4 upper=0.8 effort=70.0 velocity=6.28; origin xyz=0 0.128943749506644 0.352787572334531 rpy=0.28228151180682093 0.3786256514483699 0.1067984530673944 -> xyz=0 0.128943749506644 0.351787572334531 rpy=0.261799387799151 0 0
- joint left_shoulder_roll_joint: limit lower=-0.6 upper=2.7 effort=72 velocity=8.164 -> lower=-0.3 upper=2.7 effort=70.0 velocity=6.28; origin xyz=0 0.0630000000000002 0 rpy=-0.16179938779915 0 0 -> xyz=0 0.0629999999999999 0 rpy=-0.261799387799151 0 0
- joint left_shoulder_yaw_joint: limit lower=-3.7175512 upper=1.623156 effort=72.0 velocity=8.164 -> lower=-1.8 upper=1.8 effort=6.28 velocity=70.0; origin xyz=0 0.065813 -0.091069 rpy=0 -0.2618 1.5708 -> xyz=0 0.0658130327873276 -0.0910694499562512 rpy=0.261799387799152 0 0
- joint left_wrist_pitch_joint: limit lower=-1.05 upper=1.05 effort=30 velocity=6.28 -> lower=-1.05 upper=1.05 effort=30.0 velocity=6.28; origin xyz=0 0 -0.065 rpy=0 0 0 -> xyz=0 0 -0.0650000000000001 rpy=0 0 0
- joint left_wrist_roll_joint: limit lower=-1.11 upper=1.11 effort=30 velocity=6.28 -> lower=-1.11 upper=1.11 effort=30.0 velocity=6.28; origin xyz=0 0.00025882 -0.064034 rpy=0 0 0 -> xyz=0 0 -0.0649999999999999 rpy=0 0 0
- joint left_wrist_yaw_joint: limit lower=-1.1519173 upper=4.043510 effort=30 velocity=6.28 -> lower=-1.57 upper=1.57 effort=30.0 velocity=6.28; origin xyz=0 0 -0.0915 rpy=0 0 -1.5708 -> xyz=0 0 -0.0915 rpy=0 0 0
- joint right_ankle_pitch_joint: limit lower=-0.7 upper=0.95 effort=72 velocity=12.0 -> lower=-0.7 upper=0.95 effort=72.0 velocity=12.0; origin xyz=0.000178827472855806 0 -0.36737068203755 rpy=0 0 0 -> xyz=0 0 -0.371366732487818 rpy=0 0 0
- joint right_ankle_roll_joint: axis 0.996194698091745 0 -0.0871557427476598 -> 0.996194698091743 0 -0.0871557427476899; limit lower=-0.45 upper=0.45 effort=72 velocity=12.0 -> lower=-0.45 upper=0.45 effort=72.0 velocity=12.0; origin xyz=0 0 0 rpy=0 -0.0428243667780054 0 -> xyz=0 0 0 rpy=0 -0.042824366778005 0
- joint right_elbow_joint: limit lower=0.0 upper=2.17 effort=72 velocity=8.164 -> lower=0.0 upper=2.17 effort=70.0 velocity=6.28; origin xyz=0 0.00025881904510261 -0.151965925826289 rpy=1.04720 0 0 -> xyz=0 0 -0.151 rpy=0 0 0
- joint right_hip_pitch_joint: limit lower=-1.57 upper=1.57 effort=320 velocity=12.0 -> lower=-1.5708 upper=1.5708 effort=320.0 velocity=12.0; origin xyz=0 0.00680000000000022 -0.1652 rpy=0 0 0 -> xyz=0 0.00680000000000042 -0.165200000000001 rpy=0 0 0
- joint right_hip_roll_joint: limit lower=-1.57 upper=0.25 effort=300 velocity=12.0 -> lower=-1.5708 upper=0.1 effort=320.0 velocity=12.0
- joint right_hip_yaw_joint: limit lower=-1.57 upper=1.57 effort=90 velocity=12.0 -> lower=-1.5708 upper=1.5708 effort=90.0 velocity=12.0
- joint right_knee_joint: limit lower=0.0 upper=2.36 effort=320 velocity=12.0 -> lower=0.0 upper=2.356 effort=320.0 velocity=12.0; origin xyz=0 0 -0.380000000000003 rpy=0 0 0 -> xyz=0 0 -0.38 rpy=0 0 0
- joint right_shoulder_pitch_joint: limit lower=-1.2 upper=2.4 effort=72 velocity=8.164 -> lower=-0.8 upper=2.4 effort=70.0 velocity=6.28; origin xyz=0 -0.128943749506644 0.352787572334531 rpy=-0.28228151180682093 0.3786256514483699 -0.1067984530673944 -> xyz=0 -0.128943749506644 0.351787572334532 rpy=-0.261799387799149 0 0
- joint right_shoulder_roll_joint: limit lower=-2.7 upper=0.6 effort=72 velocity=8.164 -> lower=-2.7 upper=0.3 effort=70.0 velocity=6.28; origin xyz=0 -0.063 0 rpy=0.16179938779915 0 0 -> xyz=0 -0.063 0 rpy=0.261799387799149 0 0
- joint right_shoulder_yaw_joint: limit lower=-1.623156 upper=3.7175512 effort=72 velocity=8.164 -> lower=-1.8 upper=1.8 effort=70.0 velocity=6.28; origin xyz=0 -0.065813 -0.091069 rpy=0 -0.2618 -1.5708 -> xyz=0 -0.0658130327873273 -0.0910694499562514 rpy=-0.261799387799149 0 0
- joint right_wrist_pitch_joint: limit lower=-1.05 upper=1.05 effort=30 velocity=6.28 -> lower=-1.05 upper=1.05 effort=30.0 velocity=6.28; origin xyz=0 0 -0.065 rpy=0 0 0 -> xyz=0 0 -0.0649999999999999 rpy=0 0 0
- joint right_wrist_roll_joint: limit lower=-1.11 upper=1.11 effort=30 velocity=6.28 -> lower=-1.11 upper=1.11 effort=30.0 velocity=6.28; origin xyz=0 -0.00025882 -0.064034 rpy=0 0 0 -> xyz=0 0 -0.0650000000000002 rpy=0 0 0
- joint right_wrist_yaw_joint: limit lower=-4.043510 upper=1.1519173 effort=30 velocity=6.28 -> lower=-1.57 upper=1.57 effort=30.0 velocity=6.28; origin xyz=0 0 -0.0915 rpy=0 0 1.5708 -> xyz=0 0 -0.0915 rpy=0 0 0
- joint waist_yaw_joint: limit lower=-2.62 upper=2.62 effort=150 velocity=6.28 -> lower=-2.618 upper=2.618 effort=150.0 velocity=6.28
