Commit message: 更加手部的碰撞体积

File: source/unitree_rl_lab/unitree_rl_lab/assets/robots/humanoid_ultra_description/urdf/humanoid_ultra_27dof_description.urdf (robot description, URDF)
Before this commit: robot humanoidultra01, 28 links, 27 joints
Links:
- link left_wrist_pitch_link: geometry collision mesh filename=package://humanoidultra01/meshes/left_wrist_pitch_link.STL scale=1.1 1.1 1.1; visual mesh filename=package://humanoidultra01/meshes/left_wrist_pitch_link.STL
- link right_wrist_pitch_link: geometry collision mesh filename=package://humanoidultra01/meshes/right_wrist_pitch_link.STL scale=1.1 1.1 1.1; visual mesh filename=package://humanoidultra01/meshes/right_wrist_pitch_link.STL
